File: Onboarding.kicad_sch (KiCad schematic)
At the start: 0 parts

Commit message: Test Commit
Parts:
- added C1: 100u, symbol Device:C
- added R1: 180, symbol Device:R
- added RSC: .22, symbol Device:R
- added U2: MC34063A, Package_SO:SOIC-8_3.9x4.9mm_P1.27mm, symbol ! Robomaster ICs:MC34063A

Commit message: Update Onboarding.kicad_sch
Parts:
- added 330u: C_Polarized, symbol Device:C_Polarized
- added C2: 1500p, symbol Device:C
- added D1: 1N5819, Diode_THT:D_DO-41_SOD81_P10.16mm_Horizontal, symbol Diode:1N5819
- added L1: 170u, symbol Device:L_Iron
- added R2: 2.2k, symbol Device:R
- added R3: 47k, symbol Device:R
Connections:
- net at U2.1 (SC): now also D1.2 (A), L1.2
- net GND: now reaches U2.2 (SE)
- net GND: now also C1.2, U2.4 (GND), 330u.2, C2.2, R2.2
- net at U2.3 (CT): now also C2.1
- net at U2.5 (COMP-): now also R2.1, R3.1
- net +12V: now reaches U2.6 (VCC)
- net +12V: now also C1.1, RSC.2
- net at U2.7 (I_{PK}): now also R1.1, RSC.1, L1.1
- net at U2.8 (DC): now also R1.2
- new net VOUT: 330u.1, D1.1 (K), R3.2
Other:
- moved on the sheet: C1, R1, RSC, U2

Commit message: Finish Schematic
Parts:
- removed 330u: C_Polarized, symbol Device:C_Polarized
- removed RSC: .22, symbol Device:R
- added C3: 330u, Capacitor_SMD:C_0805_2012Metric, symbol Device:C_Polarized
- added H1, H2, H3, H4: MountingHole, MountingHole:MountingHole_2.2mm_M2, symbol Mechanical:MountingHole
- added J1: Conn_01x02, Connector_AMASS:AMASS_XT30U-F_1x02_P5.0mm_Vertical, symbol Connector_Generic:Conn_01x02
- added J2: Conn_01x02, Connector_AMASS:AMASS_XT30U-M_1x02_P5.0mm_Vertical, symbol Connector_Generic:Conn_01x02
- added J3, J4: Conn_01x02, Connector_JST:JST_GH_BM02B-GHS-TBT_1x02-1MP_P1.25mm_Vertical, symbol Connector_Generic:Conn_01x02
- added R4: .22, Resistor_SMD:R_0603_1608Metric_Pad0.98x0.95mm_HandSolder, symbol Device:R
- added TP1: VC, TestPoint:TestPoint_Bridge_Pitch2.0mm_Drill0.7mm, symbol Connector:TestPoint
- added TP2: VE, TestPoint:TestPoint_Bridge_Pitch2.0mm_Drill0.7mm, symbol Connector:TestPoint
- added V1: 12, symbol Simulation_SPICE:VDC
- C1: footprint (none) -> Capacitor_THT:CP_Radial_D8.0mm_P5.00mm
- C2: footprint (none) -> Capacitor_SMD:C_0603_1608Metric_Pad1.08x0.95mm_HandSolder
- D1: footprint Diode_THT:D_DO-41_SOD81_P10.16mm_Horizontal -> Diode_SMD:D_SOD-123F
- L1: footprint (none) -> Inductor_SMD:L_6.3x6.3_H3
- R1: footprint (none) -> Resistor_SMD:R_0805_2012Metric_Pad1.20x1.40mm_HandSolder
- R2, R3: footprint (none) -> Resistor_SMD:R_0603_1608Metric_Pad0.98x0.95mm_HandSolder
Connections:
- net +12V: now also J1.1 (Pin_1), R4.2, V1.1
- net GND: now also C3.2, J1.2 (Pin_2), J2.2 (Pin_2), V1.2
- net at D1.2 (A), L1.2, U2.1 (SC): now also TP2.1
- net at L1.1, R1.1, U2.7 (I_{PK}): now also R4.1, TP1.1
- net VOUT renamed VCC
- net VCC: now also C3.1, J2.1 (Pin_1)
- new net CAN+: J3.1 (Pin_1), J4.1 (Pin_1)
- new net CAN-: J3.2 (Pin_2), J4.2 (Pin_2)
Other:
- note added: "12V to 28V 0.175mA Boost Converter"
- note added: "CAN Connections"
- note added: "Input Power"
- note added: "Mounting Holes"
- note added: "Output Power"
- note added: "SPICE Simulation Input Voltage"
