File: Onboarding.kicad_sch (KiCad schematic)
At the start: 0 parts

Commit message: commit ethanchu
Parts:
- added C1: 330u, Capacitor_THT:CP_Radial_D8.0mm_P5.00mm, symbol Device:C
- added C2: 100u, Capacitor_SMD:C_0805_2012Metric, symbol Device:C
- added C3: 1500p, Capacitor_SMD:C_0603_1608Metric_Pad1.08x0.95mm_HandSolder, symbol Device:C
- added D1: 1N5819, Diode_THT:D_DO-41_SOD81_P10.16mm_Horizontal, symbol Diode:1N5819
- added H1, H2, H3, H4: MountingHole, MountingHole:MountingHole_2.2mm_M2, symbol Mechanical:MountingHole
- added J1: Conn_01x02, Connector_AMASS:AMASS_XT30U-F_1x02_P5.0mm_Vertical, symbol Connector_Generic:Conn_01x02
- added J2: Conn_01x02, Connector_AMASS:AMASS_XT30U-M_1x02_P5.0mm_Vertical, symbol Connector_Generic:Conn_01x02
- added J3, J4: Conn_01x02, Connector_JST:JST_GH_BM02B-GHS-TBT_1x02-1MP_P1.25mm_Vertical, symbol Connector_Generic:Conn_01x02
- added L1: 170u, RM_Example:INDM3225X240N, symbol Device:L
- added R1: 2.2K, Resistor_SMD:R_0603_1608Metric_Pad0.98x0.95mm_HandSolder, symbol Device:R
- added R2: 47K, Resistor_SMD:R_0603_1608Metric_Pad0.98x0.95mm_HandSolder, symbol Device:R
- added R3: 0.22, Resistor_SMD:R_0603_1608Metric_Pad0.98x0.95mm_HandSolder, symbol Device:R
- added R4: 180, Resistor_SMD:R_0805_2012Metric_Pad1.20x1.40mm_HandSolder, symbol Device:R
- added TP1: Vc, TestPoint:TestPoint_Bridge_Pitch2.0mm_Drill0.7mm, symbol Connector:TestPoint
- added TP2: Ve, TestPoint:TestPoint_Bridge_Pitch2.0mm_Drill0.7mm, symbol Connector:TestPoint
- added U1: MC34063A, Package_SO:SOIC-8_3.9x4.9mm_P1.27mm, symbol RM_IC:MC34063A
- added V1: 12, symbol Simulation_SPICE:VDC
Connections:
- new net: L1.1, R3.1, R4.1, TP1.1, U1.7 (I_{PK})
- new net: D1.2 (A), L1.2, TP2.1, U1.1 (SC)
- new net: R1.1, R2.1, U1.5 (COMP-)
- new net: C3.1, U1.3 (CT)
- new net: R4.2, U1.8 (DC)
- new net +12V: C2.1, J1.2 (Pin_2), R3.2, U1.6 (VCC), V1.1
- new net CAN+: J3.2 (Pin_2), J4.2 (Pin_2)
- new net CAN-: J3.1 (Pin_1), J4.1 (Pin_1)
- new net GND: C1.2, C2.2, C3.2, J1.1 (Pin_1), J2.1 (Pin_1), R1.2, U1.2 (SE), U1.4 (GND), V1.2
- new net Vout: C1.1, D1.1 (K), J2.2 (Pin_2), R2.2

Commit message: Ethan_Chu
Parts:
- D1: footprint Diode_THT:D_DO-41_SOD81_P10.16mm_Horizontal -> RM_Example:SOD3716X145N
- L1: footprint RM_Example:INDM3225X240N -> RM_Example:SPT30L174MLD
Changed lines of the file:
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@@
 			)
 		)
-		(property "Footprint" "RM_Example:INDM3225X240N"
+		(property "Footprint" "RM_Example:SPT30L174MLD"
 			(at 130.81 68.58 0)
 			(effects
@@
 			)
 		)
-		(property "Footprint" "Diode_THT:D_DO-41_SOD81_P10.16mm_Horizontal"
+		(property "Footprint" "RM_Example:SOD3716X145N"
 			(at 160.655 88.9 0)
 			(effects

Commit message: Ethan_Chu
Connections:
- net Vc: now reaches L1.1, R3.1, R4.1, TP1.1, U1.7 (I_{PK})
- net Ve: now reaches D1.2 (A), L1.2, TP2.1, U1.1 (SC)
- net V5: now reaches R1.1, R2.1, U1.5 (COMP-)
Changed lines of the file:
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@@
+		)
+	)
+	(global_label "V5"
+		(shape input)
+		(at 114.3 104.14 180)
+		(fields_autoplaced yes)
+		(effects
+			(font
+				(size 1.27 1.27)
+			)
+			(justify right)
+		)
+		(property "Intersheetrefs" "${INTERSHEET_REFS}"
+			(at 109.0167 104.14 0)
+			(effects
+				(font
+					(size 1.27 1.27)
+				)
+				(justify right)
+				(hide yes)
+			)
+		)
+	)
+	(global_label "Vc"
+		(shape input)
+		(at 107.95 68.58 180)
+		(fields_autoplaced yes)
+		(effects
+			(font
+				(size 1.27 1.27)
+			)
+			(justify right)
+		)
+		(property "Intersheetrefs" "${INTERSHEET_REFS}"
+			(at 102.7876 68.58 0)
+			(effects
+				(font
+					(size 1.27 1.27)
+				)
+				(justify right)
+				(hide yes)
+			)
+		)
+	)
+	(global_label "Ve"
+		(shape input)
+		(at 156.21 68.58 0)
+		(fields_autoplaced yes)
+		(effects
+			(font
+				(size 1.27 1.27)
+			)
+			(justify left)
+		)
+		(property "Intersheetrefs" "${INTERSHEET_REFS}"
+			(at 161.3724 68.58 0)
+			(effects
+				(font
+					(size 1.27 1.27)
+				)
+				(justify left)
+				(hide yes)
+			)
 		)
 	)
