File: Onboarding.kicad_pcb (KiCad board)
At the start: 2 copper layers, 40 x 30 mm, 20 parts, among them J1 Conn_01x02, J2 Conn_01x02, J3 Conn_01x02, J4 Conn_01x02, U2 MC34063A

Commit message: updated onboarding
Routing:
- net +12V: track 31.0 -> 32.1 mm
Changed lines of the file:
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@@
 	)
 	(segment
-		(start 87 96)
-		(end 87 99.45)
+		(start 87.55 100)
+		(end 88.5 100.95)
 		(width 0.2)
 		(layer "F.Cu")
@@
 	)
 	(segment
-		(start 87 99.45)
-		(end 88.5 100.95)
+		(start 86 97)
+		(end 86 99)
+		(width 0.2)
+		(layer "F.Cu")
+		(net 4)
+	)
+	(segment
+		(start 86 99)
+		(end 87 100)
+		(width 0.2)
+		(layer "F.Cu")
+		(net 4)
+	)
+	(segment
+		(start 89 94)
+		(end 86 97)
 		(width 0.2)
 		(layer "F.Cu")
@@
 		(start 88.5 100.95)
 		(end 91.9625 100.95)
-		(width 0.2)
-		(layer "F.Cu")
-		(net 4)
-	)
-	(segment
-		(start 89 94)
-		(end 87 96)
 		(width 0.2)
 		(layer "F.Cu")
@@
 	)
 	(segment
+		(start 87 100)
+		(end 87.55 100)
+		(width 0.2)
+		(layer "F.Cu")
+		(net 4)
+	)
+	(segment
 		(start 92 100.9125)
 		(end 94.0935 103.006)
@@
 		(start 117 95.08)
 		(end 117 96.635634)
-		(width 0.2)
-		(layer "F.Cu")
-		(net 5)
-	)
-	(segment
-		(start 115.635634 98)
-		(end 115 98)
 		(width 0.2)
 		(layer "F.Cu")
@@
 	)
 	(segment
-		(start 109.475 102.405)
-		(end 110.595 102.405)
-		(width 0.2)
-		(layer "F.Cu")
-		(net 5)
-	)
-	(segment
 		(start 103.57 90)
 		(end 103.57 90.413134)
@@
 	)
 	(segment
-		(start 117 96.635634)
-		(end 115.635634 98)
-		(width 0.2)
-		(layer "F.Cu")
-		(net 5)
-	)
-	(segment
 		(start 111 94.5)
 		(end 116.42 94.5)
-		(width 0.2)
-		(layer "F.Cu")
-		(net 5)
-	)
-	(segment
-		(start 110.595 102.405)
-		(end 115 98)
 		(width 0.2)
 		(layer "F.Cu")
@@
 		(width 0.2)
 		(layer "F.Cu")
+		(net 5)
+	)
+	(segment
+		(start 111.230634 102.405)
+		(end 109.475 102.405)
+		(width 0.2)
+		(layer "F.Cu")
+		(net 5)
+	)
+	(segment
+		(start 117 96.635634)
+		(end 111.230634 102.405)
+		(width 0.2)
+		(layer "F.Cu")

Commit message: fixed onboarding
Parts:
- D2: footprint Diode_THT:D_DO-41_SOD81_P10.16mm_Horizontal -> Diode_SMD:D_0805_2012Metric
- moved D2 9.61 mm to (110.5, 92.0), turned to 0 degrees
- moved R2 8.02 mm to (107.0, 86.0), turned to 90 degrees
- moved C2 3.64 mm to (116.0, 97.0), turned to 0 degrees
- moved J3 3.50 mm to (88.5, 87.0), turned to 180 degrees
- moved C1 2.06 mm to (110.1, 85.5)
- moved J4 2.00 mm to (90.5, 79.5), turned to 180 degrees
- moved TP1 1.80 mm to (109.5, 95.5), turned to 0 degrees
- moved U2 1.12 mm to (108.0, 100.0)
Routing:
- net +12V: track 32.1 -> 0.00 mm
- net Net-(U2-COMP-): track 8.15 -> 24.1 mm
- net Net-(U2-I_{PK}): track 23.6 -> 7.83 mm
- net VCC: track 25.7 -> 18.0 mm
- net Net-(D2-A): track 29.7 -> 23.0 mm
- net /CAN-: track 15.0 -> 8.66 mm
- net /CAN+: track 13.6 -> 8.66 mm
- net Net-(U2-CT): track 3.44 -> 5.64 mm
- net Net-(U2-DC): track 10.8 -> 11.6 mm
- added copper zone on F.Cu, net +12V
- added copper zone on F.Cu, net Net-(U2-I_{PK})

Commit message: fixed 90 degree angle
Routing:
- net Net-(U2-COMP-): track 24.1 -> 23.5 mm
Changed lines of the file:
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@@
 	)
 	(segment
-		(start 101.5 84)
-		(end 101.5 98.0875)
+		(start 105.9125 84)
+		(end 102.5 84)
+		(width 0.5)
+		(layer "F.Cu")
+		(net 10)
+	)
+	(segment
+		(start 102.5 84)
+		(end 101.5 85)
 		(width 0.5)
 		(layer "F.Cu")
@@
 	)
 	(segment
-		(start 105.9125 84)
-		(end 101.5 84)
+		(start 101.5 85)
+		(end 101.5 98.0875)
 		(width 0.5)
 		(layer "F.Cu")
