File: OnboardingBoard.kicad_pcb (KiCad board)
At the start: 2 copper layers, 44 x 37 mm, 20 parts, among them J1 Conn_01x02, J2 Conn_01x02, J3 Conn_01x02, J4 Conn_01x02, U2 MC34063A

Commit message: UpdatePCB
Parts:
- moved J2 2.00 mm to (97.0, 100.0)
- moved C4 1.05 mm to (129.0, 102.0)
- moved R4 1.00 mm to (113.4, 104.0)
- moved R5 1.00 mm to (131.5, 98.0), turned to -90 degrees
- moved C2 0.62 mm to (113.0, 99.0)
- moved J1 0.50 mm to (132.5, 83.5)
Routing:
- net Net-(U2-I_{PK}): track 66.1 -> 19.7 mm
- net GND: track 23.8 -> 0.00 mm
- net Net-(D1-A): track 35.4 -> 20.6 mm
- net VCC: track 23.9 -> 10.8 mm
- net +12V: track 23.4 -> 20.8 mm
- net Net-(U2-COMP-): track 10.8 -> 12.2 mm
- added copper zone on F.Cu, net (none)
- added copper zone on F.Cu, net Net-(U2-I_{PK})
- added copper zone on F.Cu, net VCC
